File: ArithmeticLogicUnit.kicad_sch (KiCad schematic)
At the start: 50 parts, among them U10 74LS86, U11 74HC00, U12 74LS08, U13 74HC32, U14 74LS86, U15 74LS08, U16 74HC32, U17 74LS86, U18 74LS86, U19 74LS11, U34 74LS688, U35 74LS541, U36 74LS283, U37 74LS377, U38 74LS541, U39 74HC151, U40 74LS138, U41 74LS377, U42 74LS541, U43 74LS157, U44 74LS540, U45 74LS173, U46 74LS283, U47 74LS541, U48 74LS541

Commit message: Cleans up and restructures schematics
Connections:
- net ALU_OP_0: now also U39.11 (S0)
- net ALU_OP_1: now also U39.10 (S1)
- net ALU_OP_2: now also U39.9 (S2)
- net RESET: now also U45.15 (Mr)
- net /RESET: no longer U45.15 (Mr)
- net /SHR_OUT: now also U42.19 (G2)

Commit message: Fixes Gate symbol refs and adds backplane definition
Parts:
- removed U10, U14, U17, U18: 74LS86, Package_DIP:DIP-14_W7.62mm, symbol 74xx:74LS86
- removed U11: 74HC00, Package_DIP:DIP-14_W7.62mm, symbol 74xx:74HC00
- removed U12, U15: 74LS08, Package_DIP:DIP-14_W7.62mm, symbol 74xx:74LS08
- removed U13, U16: 74HC32, Package_DIP:DIP-14_W7.62mm, symbol 74-Series:74HC32
- removed U19: 74LS11, Package_DIP:DIP-14_W7.62mm, symbol 74xx:74LS11
- added U1, U2: 74LS32, symbol 74xx:74LS32
- added U10: 74LS00, symbol 74xx:74LS00
- added U3, U4, U7, U8: 74LS86, symbol 74xx:74LS86
- added U5, U6: 74LS08, symbol 74xx:74LS08
- added U9: 74LS11, symbol 74xx:74LS11
- renumbered C31 to C?, C27 to C?, C34 to C?, C26 to C?, C15 to C?, C35 to C?, C25 to C?, C12 to C?, C28 to C?, C11 to C?, C19 to C?, C29 to C?, C10 to C?, C14 to C?, C13 to C?, C23 to C?, C18 to C?, C30 to C?, C16 to C?, C20 to C?, C32 to C?, C21 to C?, C17 to C?, C24 to C?, C22 to C?, U34 to U?, U35 to U?, U36 to U?, U37 to U?, U38 to U?, U39 to U?, U40 to U?, U41 to U?, U42 to U?, U43 to U?, U44 to U?, U45 to U?, U46 to U?, U47 to U?, U48 to U?
Connections:
- net ADDH_C: now also U10.10, U10.9
- net AND_0: now also U5.3
- net AND_1: now also U5.6
- net AND_2: now also U5.8
- net AND_3: now also U5.11
- net AND_4: now also U6.3
- net AND_5: now also U6.6
- net AND_6: now also U6.8
- net AND_7: now also U6.11
- net GND: now also U1.7 (GND), U10.7 (GND), U2.7 (GND), U3.7 (GND), U4.7 (GND), U5.7 (GND), U6.7 (GND), U7.7 (GND), U8.7 (GND), U9.10, U9.11, U9.3, U9.4, U9.5, U9.7 (GND), U9.9
- net OR_0: now also U1.3
- net OR_1: now also U1.6
- net OR_2: now also U1.8
- net OR_3: now also U1.11
- net OR_4: now also U2.3
- net OR_5: now also U2.6
- net OR_6: now also U2.8
- net OR_7: now also U2.11
- net RESET: now also U10.4, U10.5
- net SUB: now also U10.11, U7.10, U7.13, U7.2, U7.5, U8.10, U8.13, U8.2, U8.5
- net SUB_0: now also U7.3
- net SUB_1: now also U7.6
- net SUB_2: now also U7.8
- net SUB_3: now also U7.11
- net SUB_4: now also U8.3
- net SUB_5: now also U8.6
- net SUB_6: now also U8.8
- net SUB_7: now also U8.11
- net VCC: now also U1.14 (VCC), U10.1, U10.14 (VCC), U10.2, U2.14 (VCC), U3.14 (VCC), U4.14 (VCC), U5.14 (VCC), U6.14 (VCC), U7.14 (VCC), U8.14 (VCC), U9.14 (VCC)
- net XOR_0: now also U3.3
- net XOR_1: now also U3.6
- net XOR_2: now also U3.8
- net XOR_3: now also U3.11
- net XOR_4: now also U4.3
- net XOR_5: now also U4.6
- net XOR_6: now also U4.8
- net XOR_7: now also U4.11
- net X_0: now also U1.1, U3.1, U5.1
- net X_1: now also U1.4, U3.4, U5.4
- net X_2: now also U1.9, U3.9, U5.9
- net X_3: now also U1.12, U3.12, U5.12
- net X_4: now also U2.1, U4.1, U6.1
- net X_5: now also U2.4, U4.4, U6.4
- net X_6: now also U2.9, U4.9, U6.9
- net X_7: now also U2.12, U4.12, U6.12
- net Y_0: now also U1.2, U3.2, U5.2, U7.1
- net Y_1: now also U1.5, U3.5, U5.5, U7.4
- net Y_2: now also U1.10, U3.10, U5.10, U7.9
- net Y_3: now also U1.13, U3.13, U5.13, U7.12
- net Y_4: now also U2.2, U4.2, U6.2, U8.1
- net Y_5: now also U2.5, U4.5, U6.5, U8.4
- net Y_6: now also U2.10, U4.10, U6.10, U8.9
- net Y_7: now also U2.13, U4.13, U6.13, U8.12
- net /ADDH_C: now also U10.8
- net /ADD_OUT: now also U9.12
- net /RESET: now also U10.6
- net /SEL_ADD: now also U9.1
- net /SEL_CMP: now also U10.13, U9.13
- net /SEL_SUB: now also U10.12, U9.2
