File: MemoryUnit.kicad_sch (KiCad schematic)
At the start: 21 parts, among them U20 CY62256-70PC, U21 74LS30, U22 74LS32, U49 74LS377, U50 74LS30, U51 74LS138, U52 74LS377, U53 74LS377, U54 74HC541, U55 74HC541, U56 74LS377

Commit message: Cleans up and restructures schematics
Connections:
- net GND: now also U52.10 (GND), U54.1 (~{OE}1), U55.1 (~{OE}1)
Changed lines of the file:
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@@
 			)
 		)
-		(property "Function" "MARLO"
-			(at 204.0733 30.48 0)
-			(effects
-				(font
-					(size 1.27 1.27)
-				)
-			)
-		)
 		(property "Value" "74LS377"
 			(at 204.0733 35.56 0)
@@
 			)
 		)
+		(property "Function" "MARLO"
+			(at 204.0733 30.48 0)
+			(effects
+				(font
+					(size 1.27 1.27)
+				)
+			)
+		)
 		(pin "1"
 		)
@@
 	)
 	(symbol
+		(lib_id "power:GND")
+		(at 31.75 128.27 270)
+		(unit 1)
+		(exclude_from_sim no)
+		(in_bom yes)
+		(on_board yes)
+		(dnp no)
+		(fields_autoplaced yes)
+		(property "Reference" "#PWR473"
+			(at 38.1 128.27 0)
+			(effects
+				(font
+					(size 1.27 1.27)
+				)
+				(hide yes)
+			)
+		)
+		(property "Value" "GND"
+			(at 35.56 128.27 90)
+			(effects
+				(font
+					(size 1.27 1.27)
+				)
+				(justify right)
+			)
+		)
+		(property "Footprint" ""
+			(at 31.75 128.27 0)
+			(effects
+				(font
+					(size 1.27 1.27)
+				)
+				(hide yes)
+			)
+		)
+		(property "Datasheet" ""
+			(at 31.75 128.27 0)
+			(effects
+				(font
+					(size 1.27 1.27)
+				)
+				(hide yes)
+			)
+		)
+		(property "Description" "Power symbol creates a global label with name \"GND\" , ground"
+			(at 31.75 128.27 0)
+			(effects
+				(font
+					(size 1.27 1.27)
+				)
+				(hide yes)
+			)
+		)
+		(pin "1"
+		)
+		(instances
+			(project "Kestrel8"
+				(path "/afdf0bd2-bb31-4132-9ca5-f1f94e74d630/0634ef32-2c4c-48f1-8aa2-2dae2aa275c2"
+					(reference "#PWR473")
+					(unit 1)
+				)
+			)
+		)
+	)
+	(symbol
 		(lib_id "power:VCC")
 		(at 201.93 25.4 0)
@@
 	)
 	(symbol
+		(lib_id "power:GND")
+		(at 85.09 128.27 270)
+		(unit 1)
+		(exclude_from_sim no)
+		(in_bom yes)
+		(on_board yes)
+		(dnp no)
+		(fields_autoplaced yes)
+		(property "Reference" "#PWR472"
+			(at 91.44 128.27 0)
+			(effects
+				(font
+					(size 1.27 1.27)
+				)
+				(hide yes)
+			)
+		)
+		(property "Value" "GND"
+			(at 88.9 128.27 90)
+			(effects
+				(font
+					(size 1.27 1.27)
+				)
+				(justify right)
+			)
+		)
+		(property "Footprint" ""
+			(at 85.09 128.27 0)
+			(effects
+				(font
+					(size 1.27 1.27)
+				)
+				(hide yes)
+			)
+		)
+		(property "Datasheet" ""
+			(at 85.09 128.27 0)
+			(effects
+				(font
+					(size 1.27 1.27)
+				)
+				(hide yes)
+			)
+		)
+		(property "Description" "Power symbol creates a global label with name \"GND\" , ground"
+			(at 85.09 128.27 0)
+			(effects
+				(font
+					(size 1.27 1.27)
+				)
+				(hide yes)
+			)
+		)
+		(pin "1"
+		)
+		(instances
+			(project "Kestrel8"
+				(path "/afdf0bd2-bb31-4132-9ca5-f1f94e74d630/0634ef32-2c4c-48f1-8aa2-2dae2aa275c2"
+					(reference "#PWR472")
+					(unit 1)
+				)
+			)
+		)
+	)
+	(symbol
 		(lib_id "Device:C")
 		(at 104.14 93.98 90)
@@
 			)
 		)
-		(property "Function" "IO_SELECT"
-			(at 91.4317 215.90 0)
-			(effects
-				(font
-					(size 1.27 1.27)
-				)
-			)
-		)
 		(property "Value" "74LS30"
 			(at 91.4317 220.98 0)
@@
 			)
 		)
+		(property "Function" "IO_SELECT"
+			(at 91.4317 215.9 0)
+			(effects
+				(font
+					(size 1.27 1.27)
+				)
+			)
+		)
 		(pin "5"
 		)
@@
 			)
 		)
-		(property "Function" "ADR_DECODE"
-			(at 182.4833 210.82 0)
-			(effects
-				(font
-					(size 1.27 1.27)
-				)
-			)
-		)
 		(property "Value" "74LS138"
 			(at 182.4833 215.9 0)
@@
 			)
 		)
+		(property "Function" "ADR_DECODE"
+			(at 182.4833 210.82 0)
+			(effects
+				(font
+					(size 1.27 1.27)
+				)
+			)
+		)
 		(pin "13"
 		)
@@
 			)
 		)
-		(property "Function" "MARHI"
-			(at 257.4133 30.48 0)
-			(effects
-				(font
-					(size 1.27 1.27)
-				)
-			)
-		)
 		(property "Value" "74LS377"
 			(at 257.4133 35.56 0)
@@
 			)
 		)
+		(property "Function" "MARHI"
+			(at 257.4133 30.48 0)
+			(effects
+				(font
+					(size 1.27 1.27)
+				)
+			)
+		)
 		(pin "1"
 		)
@@
 			)
 		)
-		(property "Function" "TLO"
-			(at 46.5933 30.48 0)
-			(effects
-				(font
-					(size 1.27 1.27)
-				)
-			)
-		)
 		(property "Value" "74LS377"
 			(at 46.5933 35.56 0)
@@
 			)
 		)
+		(property "Function" "TLO"
+			(at 46.5933 30.48 0)
+			(effects
+				(font
+					(size 1.27 1.27)
+				)
+			)
+		)
 		(pin "1"
 		)
@@
 			)
 		)
-		(property "Function" "THI_OUTPUT"
-			(at 99.9333 95.25 0)
-			(effects
-				(font
-					(size 1.27 1.27)
-				)
-			)
-		)
 		(property "Value" "74HC541"
 			(at 99.9333 100.33 0)
@@
 			)
 		)
+		(property "Function" "THI_OUTPUT"
+			(at 99.9333 95.25 0)
+			(effects
+				(font
+					(size 1.27 1.27)
+				)
+			)
+		)
 		(pin "6"
 		)
@@
 	)
 	(symbol
+		(lib_id "power:GND")
+		(at 255.27 73.66 0)
+		(unit 1)
+		(exclude_from_sim no)
+		(in_bom yes)
+		(on_board yes)
+		(dnp no)
+		(fields_autoplaced yes)
+		(property "Reference" "#PWR474"
+			(at 261.62 73.66 0)
+			(effects
+				(font
+					(size 1.27 1.27)
+				)
+				(hide yes)
+			)
+		)
+		(property "Value" "GND"
+			(at 259.08 73.66 90)
+			(effects
+				(font
+					(size 1.27 1.27)
+				)
+				(justify right)
+			)
+		)
+		(property "Footprint" ""
+			(at 255.27 73.66 0)
+			(effects
+				(font
+					(size 1.27 1.27)
+				)
+				(hide yes)
+			)
+		)
+		(property "Datasheet" ""
+			(at 255.27 73.66 0)
+			(effects
+				(font
+					(size 1.27 1.27)
+				)
+				(hide yes)
+			)
+		)
+		(property "Description" "Power symbol creates a global label with name \"GND\" , ground"
+			(at 255.27 73.66 0)
+			(effects
+				(font
+					(size 1.27 1.27)
+				)
+				(hide yes)
+			)
+		)
+		(pin "1"
+		)
+		(instances
+			(project "Kestrel8"
+				(path "/afdf0bd2-bb31-4132-9ca5-f1f94e74d630/0634ef32-2c4c-48f1-8aa2-2dae2aa275c2"
+					(reference "#PWR474")
+					(unit 1)
+				)
+			)
+		)
+	)
+	(symbol
 		(lib_id "74xx:74LS32")
 		(at 322.58 171.45 0)
@@
 			)
 		)
-		(property "Function" "TLO_OUTPUT"
-			(at 46.5933 95.25 0)
-			(effects
-				(font
-					(size 1.27 1.27)
-				)
-			)
-		)
 		(property "Value" "74HC541"
 			(at 46.5933 100.33 0)
@@
 			)
 		)
+		(property "Function" "TLO_OUTPUT"
+			(at 46.5933 95.25 0)
+			(effects
+				(font
+					(size 1.27 1.27)
+				)
+			)
+		)
 		(pin "6"
 		)
@@
 			)
 		)
-		(property "Function" "THI"
-			(at 99.9333 30.48 0)
-			(effects
-				(font
-					(size 1.27 1.27)
-				)
-			)
-		)
 		(property "Value" "74LS377"
 			(at 99.9333 35.56 0)
@@
 			)
 		)
+		(property "Function" "THI"
+			(at 99.9333 30.48 0)
+			(effects
+				(font
+					(size 1.27 1.27)
+				)
+			)
+		)

Commit message: Fixes Gate symbol refs and adds backplane definition
Parts:
- removed U21, U50: 74LS30, Package_DIP:DIP-14_W7.62mm, symbol 74xx:74LS30
- removed U22: 74LS32, Package_DIP:DIP-14_W7.62mm, symbol 74xx:74LS32
- added U1: 74LS32, symbol 74xx:74LS32
- added U2: 74LS30, symbol 74xx:74LS30
- renumbered C36 to C?, C43 to C?, C33 to C?, C39 to C?, C37 to C?, C42 to C?, C44 to C?, C38 to C?, C41 to C?, C40 to C?, U49 to U?, U51 to U?, U20 to U?, U52 to U?, U53 to U?, U54 to U?, U55 to U?, U56 to U?
Connections:
- net CLK: now also U1.2
- net GND: now also U1.10, U1.12, U1.13, U1.4, U1.5, U1.7 (GND), U1.9, U2.7 (GND)
- net MA_10: now also U2.3
- net MA_11: now also U2.4
- net MA_12: now also U2.5
- net MA_13: now also U2.6
- net MA_14: now also U2.11
- net MA_15: now also U2.12
- net MA_8: now also U2.1
- net MA_9: now also U2.2
- net VCC: now also U1.14 (VCC), U2.14 (VCC)
- net /IO_SEL: now also U2.8
- net /RAM_IN: now also U1.1
- net /RAM_WE: now also U1.3
Other:
- note added: "CONTROL LOGIC"
- note added: "MEMORY ADDRESS REGISTER"
- note added: "RANDOM ACCESS MEMORY"
- note added: "TEMPORARY REGISTER"
- moved on the sheet: C?, U?
